File: hardware/Pinball Matrix board Rev 1.kicad_pcb (KiCad board)
At the start: 2 copper layers, 100 x 100 mm, 151 parts, among them J1 B4B-XH-A, J2 B4B-XH-A, J3 Conn_01x13_Pin, J4 Conn_01x10_Pin, U1 LMV393, U2 LMV393, U3 ESP32-C6-DevKitM-Amazon, U4 74HC595D, U5 74HC595D, U6 VNQ7E100AJTR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

Commit message: Add files via upload
cleaned up some foot print errors  and changed tvs diodes on all 3 rail because of their size physically there were 0201's
Parts:
- added D10: H5VND5B, PCM_JLCPCB:D_SOD-523, F.Cu at (176.0, 72.2)
- added R28: 3kΩ, PCM_JLCPCB:R_0805, F.Cu at (151.2, 69.4)
- C16: value 100uf, 35V -> C_Polarized
- D2: value H3V3L10B -> H3V3LD5B; footprint PCM_JLCPCB:D_DFN1006-2L -> PCM_JLCPCB:D_SOD-523
- D4: value H5VL10B -> Yellow; footprint PCM_JLCPCB:D_DFN1006-2L -> PCM_JLCPCB:D_0805
- F2: value 30V 500ma -> Polyfuse
- L1, L2, L3, L4, L5: value IRLR024 -> IRLZ24
- moved C16 48.2 mm to (160.1, 54.4)
- moved U8 37.5 mm to (133.8, 115.7)
- moved R26 35.4 mm to (148.7, 86.8), turned to -90 degrees
- moved C15 34.0 mm to (159.7, 69.4)
- moved J1 34.0 mm to (157.6, 65.0)
- moved C14 34.0 mm to (156.6, 69.4)
- moved D1 29.6 mm to (149.1, 69.2)
- moved C20 28.8 mm to (145.8, 86.8), turned to -90 degrees
- moved C19 28.5 mm to (167.7, 126.1)
- moved R27 26.8 mm to (150.5, 97.8), turned to 0 degrees
- moved R33 23.3 mm to (134.7, 89.5), turned to 180 degrees
- moved D4 22.5 mm to (153.8, 69.5), turned to -90 degrees
- moved U4 19.5 mm to (143.3, 94.5), turned to -90 degrees
- moved C21 12.5 mm to (142.8, 70.4)
- moved R29 12.5 mm to (131.4, 68.6)
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Connections:
- D4 pad 1: GND -> Net-(D4-Pad1)
- D4 pad 2: VCC_5V -> +18vdc
- H1 pad 1: (no net) -> GND
- H2 pad 1: (no net) -> GND
- H3 pad 1: (no net) -> GND

Commit message: Add files via upload
 The update PBC  errors are clean
Parts:
- removed D4: Yellow, PCM_JLCPCB:D_0805
- removed R28: 3kΩ, PCM_JLCPCB:R_0805
- added F1: Polyfuse, OptoDevice:R_LDR_7x6mm_P5.1mm_Vertical, F.Cu at (152.1, 76.8)
- moved R21 7.50 mm to (123.3, 132.3)
- moved R22 7.50 mm to (121.4, 132.4)
- moved D7 0.35 mm to (121.5, 115.5)
- moved D5 0.22 mm to (121.5, 120.1)
Connections:
- U1 pad 9: (no net) -> unconnected-(U1C-Epad-Pad9)
- U2 pad 9: (no net) -> unconnected-(U2C-Epad-Pad9)
- U6 pad 17: (no net) -> +18vdc
- U7 pad 17: (no net) -> +18vdc
