File: hardware/Pinball Matrix board Rev 1.kicad_pcb (KiCad board)
At the start: 4 copper layers, 100 x 100 mm, 155 parts, among them J1 B4B-XH-A, J2 B4B-XH-A, J3 Conn_01x13_Pin, J4 Conn_01x10_Pin, U1 LMV393, U2 LMV393, U3 ESP32-C6-DevKitM-Amazon, U4 74HC595D, U5 74HC595D, U6 VNQ7E100AJTR, U7 VNQ7E100AJTR

Commit message: before PCB purchase
Parts:
- removed REF**: 10mm LOGO, 1My_Parts_ Passive:10mm LOGO
- added 10mm1: ~, 1My_Parts_ Passive:10mm LOGO, F.Cu at (154.3, 131.8)
- F1: footprint OptoDevice:R_LDR_7x6mm_P5.1mm_Vertical -> 1My_Parts_ Passive:poly fuse
- J4: footprint Connector_Molex:Molex_KK-396_A-41791-0010_1x10_P3.96mm_Vertical -> 1My_Parts_ Connectors:Molex_KK-396_A-41791-0010_1x10_P3.96mm_Vertical
- moved F1 2.43 mm to (128.4, 67.4)
- moved TP1 0.54 mm to (160.4, 136.5)
- moved TP2 0.19 mm to (165.3, 136.5)
- renumbered +5V to TP1, SDA to TP11, SCL to TP12, 3.3v to TP2, GPIO0 to TP3, GPIO1 to TP4, GPIO8 to TP5, GND to TP6, GPIO11 to TP7, GPIO12 to TP8, GPIO13 to TP9
Routing:
- net Net-(R14-Pad2): track 30.0 -> 47.1 mm, vias 2 -> 3
- net GND: track 129.3 -> 140.3 mm
Other:
- board text added: "+5V"
- board text added: "0"
- board text added: "1"
- board text added: "11"
- board text added: "12"
- board text added: "13"
- board text added: "3.3V"
- board text added: "8"
- board text added: "GND"
