File: hardware/Pinball Matrix board Rev 1.kicad_sch (KiCad schematic)
At the start: 153 parts, among them J2 B4B-XH-A, J3 B4B-XH-A, U2 ESP32-C6-DevKitM-Amazon, U3 VNQ7E100AJTR, U5 LMV393, U6 LMV393, U7 VNQ7E100AJTR, U8 74HC595D, U9 74HC595D

Commit message: Add files via upload
Made seveal additions it's close to being complete before final review
Parts:
- removed JD1: connector "d", Connector_Molex:Molex_KK-396_5273-12A_1x12_P3.96mm_Vertical, symbol Connector_Generic_MountingPin:Conn_01x24_MountingPin
- removed R32, R33: 10kΩ, PCM_JLCPCB:R_0805, symbol PCM_JLCPCB-Resistors:0805,10kΩ
- removed TP7, TP8: TestPoint_Small, symbol Connector:TestPoint_Small
- added J3: Conn_01x13_Pin, Connector_Molex:Molex_KK-396_A-41791-0013_1x13_P3.96mm_Vertical, symbol Connector:Conn_01x13_Pin
- added J4: Conn_01x10_Pin, Connector_Molex:Molex_KK-396_A-41791-0010_1x10_P3.96mm_Vertical, symbol Connector:Conn_01x10_Pin
- added R26: 10kΩ, PCM_JLCPCB:R_0805, symbol PCM_JLCPCB-Resistors:0805,10kΩ
- added TP1, TP11, TP2, TP6: TestPoint_Small, 1My_Parts_ Connectors:KEYSTONE_5015, symbol Connector:TestPoint_Small
- F2: footprint 1206 -> digikey-footprints:1206
- L1, L2, L3, L4, L5: footprint Package_TO_SOT_SMD:TO-252-2 -> Package_TO_SOT_THT:TO-220-3_Vertical
- TP12: footprint (none) -> 1My_Parts_ Connectors:KEYSTONE_5015
- TP3: renamed from TP9; footprint (none) -> 1My_Parts_ Connectors:KEYSTONE_5015
- TP4: renamed from TP10; footprint (none) -> 1My_Parts_ Connectors:KEYSTONE_5015
- TP5: renamed from TP11; footprint (none) -> 1My_Parts_ Connectors:KEYSTONE_5015
- TP7: renamed from TP13; footprint (none) -> 1My_Parts_ Connectors:KEYSTONE_5015
- TP8: renamed from TP14; footprint (none) -> 1My_Parts_ Connectors:KEYSTONE_5015
- TP9: renamed from TP15; footprint (none) -> 1My_Parts_ Connectors:KEYSTONE_5015
- U1: renamed from U5; footprint (none) -> Package_SO:SOIC-8-1EP_3.9x4.9mm_P1.27mm_EP2.29x3mm
- U2: renamed from U6; footprint (none) -> Package_SO:SOIC-8-1EP_3.9x4.9mm_P1.27mm_EP2.29x3mm
- U3: renamed from U2; footprint RF_Module:ESP32-C3-DevKitM-1 -> 1My_Parts_ MPUs:ESP32-C6-DevKit-Amazon
- U8: renamed from U10; footprint ESP32Vroom:).96 inOLED display SSD1306 -> 1My_Parts_ ICs:0.96 inOLED display SSD1306; symbol Capt Fan esp32 lib:0.96in_OLED_SSD1306 -> 1My_Basic components:0.96in_OLED_SSD1306
- renumbered C34 to C1, C23 to C10, C38 to C11, C33 to C12, C37 to C13, C10 to C14, C11 to C15, C12 to C16, C25 to C17, C24 to C18, C40 to C19, C30 to C2, C28 to C20, C29 to C21, C9 to C22, C5 to C23, C13 to C24, C6 to C25, C16 to C26, C17 to C27, C18 to C28, C19 to C29, C35 to C3, C7 to C30, C8 to C31, C26 to C32, C27 to C33, C39 to C34, C31 to C4, C36 to C5, C32 to C6, C20 to C7, C22 to C8, C21 to C9, D3 to D2, D5 to D3, D2 to D4, D22 to D5, D23 to D6, D24 to D7, D25 to D8, D4 to D9, J2 to J1, J3 to J2, R35 to R1, R84 to R10, R39 to R11, R38 to R12, R75 to R13, R76 to R14, R85 to R15, R86 to R16, R8 to R17, R9 to R18, R10 to R19, R36 to R2, R11 to R20, R3 to R21, R4 to R22, R5 to R23, R7 to R24, R37 to R25, R31 to R27, R34 to R29, R77 to R3, R59 to R30, R68 to R31, R60 to R32, R67 to R33, R71 to R34, R69 to R35, R72 to R36, R70 to R37, R12 to R38, R13 to R39, R81 to R4, R14 to R40, R15 to R41, R16 to R42, R17 to R43, R18 to R44, R19 to R45, R25 to R46, R20 to R47, R79 to R5, R26 to R58, R58 to R59, R82 to R6, R27 to R60, R28 to R61, R29 to R62, R30 to R63, R63 to R64, R64 to R65, R73 to R66, R74 to R67, R21 to R68, R22 to R69, R78 to R7, R23 to R70, R24 to R71, R83 to R8, R80 to R9, TP6 to TP10, U8 to U4, U9 to U5, U3 to U6
Connections:
- net +3V3 is gone; now on net +3.3V: C34.1, U8.2 (VCC)
- net GNDD is gone; now on net GND: L1.3 (S), L2.3 (S), L3.3 (S), L4.3 (S), L5.3 (S), R53.2, R54.2, R55.2, R56.2, R57.2
- net I2C SCL is gone; now on net I²C SCL Display: U8.3 (SLC)
- net I2C SDA is gone; now on net I²C SDA Display: U8.4 (SDA)
- net Row 3 is gone; now on net Row_3: FB3.1, R66.2
- net Row 4 is gone; now on net Row_4: FB4.1, R67.2
- net +3.3V: now also R26.2, TP2.1
- net GND: now also U8.5 (GND), U8.6 (GND), U8.7 (GND), U8.8 (GND), TP6.1
- net I²C SCL: now also TP12.1
- net I²C SDA: now also TP11.1
- net LD3: now also J4.6 (Pin_6)
- net LD4: now also J4.9 (Pin_9)
- net LD5: now also J4.10 (Pin_10)
- net LD6: now also J4.8 (Pin_8)
- net LD7: now also J4.7 (Pin_7)
- net MX1: now also J3.1 (Pin_1)
- net MX2: now also J3.2 (Pin_2), J3.3 (Pin_3)
- net MX3: now also J3.10 (Pin_10), J3.11 (Pin_11)
- net MX4: now also J3.12 (Pin_12), J3.13 (Pin_13)
- net MX5: now also J4.1 (Pin_1), J4.2 (Pin_2)
- net MX6: now also J4.3 (Pin_3), J4.4 (Pin_4)
- net MX7: now also J4.5 (Pin_5)
- net SW_0: now also J3.7 (Pin_7)
- net SW_1: now also J3.6 (Pin_6)
- net SW_2: now also J3.5 (Pin_5)
- net SW_3: now also J3.4 (Pin_4)
- net VCC_5V: now also TP1.1
- net SR /OE: now reaches U5.13 (OE#)
- net SR /OE: now also U3.11 (GPIO10), U4.13 (OE#), R26.1
- net I²C SDA Display: now reaches U3.7 (GPIO7)
- net I²C SCL Display: now reaches U3.6 (GPIO6)
Other:
- moved on the sheet: C1, C10, C11, C12, C13, C14, C15, C16, C17, C18, C19, C2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

Commit message: Add files via upload
cleaned up some foot print errors  and changed tvs diodes on all 3 rail because of their size physically there were 0201's
Parts:
- removed D4: H5VL10B, PCM_JLCPCB:D_DFN1006-2L, symbol PCM_JLCPCB-Diodes:TVS-Bi,H5VL10B
- added D10: H5VND5B, PCM_JLCPCB:D_SOD-523, symbol PCM_JLCPCB-Diodes:TVS-Bi,H5VND5B
- C16: value 100uf, 35V -> C_Polarized
- D2: value H3V3L10B -> H3V3LD5B; footprint PCM_JLCPCB:D_DFN1006-2L -> PCM_JLCPCB:D_SOD-523; symbol PCM_JLCPCB-Diodes:TVS-Bi,H3V3L10B -> PCM_JLCPCB-Diodes:TVS-Bi,H3V3LD5B; Attrition Qty 10 -> 6; LCSC C20615781 -> C20615817; Part H3V3L10B -> H3V3LD5B; Price 0.014USD -> 0.017USD; Stock 71908 -> 116939
- F1: value PTC RESET FUSE 30V 1.85A TH -> Polyfuse
- F2: value 30V 500ma -> Polyfuse
- L1, L2, L3, L4, L5: value IRLR024 -> IRLZ24; footprint Package_TO_SOT_THT:TO-220-3_Vertical -> Package_TO_SOT_SMD:TO-252-2
Connections:
- net GND: now also D10.1
- net LD3: now also J4.20 (Pin_6); no longer J4.6 (Pin_6)
- net LD4: now also J4.23 (Pin_9); no longer J4.9 (Pin_9)
- net LD5: now also J4.24 (Pin_10); no longer J4.10 (Pin_10)
- net LD6: now also J4.22 (Pin_8); no longer J4.8 (Pin_8)
- net LD7: now also J4.21 (Pin_7); no longer J4.7 (Pin_7)
- net MX5: now also J4.15 (Pin_1), J4.16 (Pin_2); no longer J4.1 (Pin_1), J4.2 (Pin_2)
- net MX6: now also J4.17 (Pin_3), J4.18 (Pin_4); no longer J4.3 (Pin_3), J4.4 (Pin_4)
- net MX7: now also J4.19 (Pin_5); no longer J4.5 (Pin_5)
- net VCC_5V: now also D10.2
Other:
- moved on the sheet: TP2

Commit message: Add files via upload
 The update PBC  errors are clean
Parts:
- F1: footprint Through Hole,P=5.1mm -> OptoDevice:R_LDR_7x6mm_P5.1mm_Vertical
- U6, U7: footprint POWERSSO-16_STM -> 1My_Parts_ ICs:SOP50P600X148-17N
Connections:
- net +18vdc: now also U6.17 (VCC=Epad), U7.17 (VCC=Epad); no longer U6.EPAD (VCC), U7.EPAD (VCC)
- net GND: now also H1.1, H2.1, H3.1
Changed lines of the file:
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@@
 	)
 	(junction
+		(at 313.69 226.06)
+		(diameter 0)
+		(color 0 0 0 0)
+	)
+	(junction
 		(at 72.39 135.89)
 		(diameter 0)
@@
 	)
 	(junction
+		(at 313.69 231.14)
+		(diameter 0)
+		(color 0 0 0 0)
+	)
+	(junction
 		(at 48.26 121.92)
 		(diameter 0)
@@
 	(wire
 		(pts
+			(xy 313.69 220.98) (xy 313.69 226.06)
+		)
+		(stroke
+			(width 0)
+			(type default)
+		)
+	)
+	(wire
+		(pts
 			(xy 46.99 77.47) (xy 46.99 78.74)
 		)
@@
 	(wire
 		(pts
+			(xy 313.69 236.22) (xy 313.69 231.14)
+		)
+		(stroke
+			(width 0)
+			(type default)
+		)
+	)
+	(wire
+		(pts
 			(xy 260.35 232.41) (xy 255.27 232.41)
 		)
@@
 	(wire
 		(pts
+			(xy 313.69 226.06) (xy 313.69 231.14)
+		)
+		(stroke
+			(width 0)
+			(type default)
+		)
+	)
+	(wire
+		(pts
 			(xy 54.61 173.99) (xy 71.12 173.99)
 		)
@@
 	(wire
 		(pts
-			(xy 144.78 177.8) (xy 138.43 177.8)
+			(xy 138.43 177.8) (xy 144.78 177.8)
 		)
 		(stroke
@@
 		(pin "4"
 		)
+		(pin "9"
+		)
 		(instances
 			(project ""
@@
 	)
 	(symbol
+		(lib_name "LMV393_1")
 		(lib_id "Comparator:LMV393")
 		(at 140.97 170.18 0)
@@
 		(dnp no)
 		(property "Reference" "U2"
-			(at 138.684 170.18 0)
+			(at 139.446 169.672 0)
 			(effects
 				(font
 					(size 1.27 1.27)
 				)
-				(justify left)
 			)
 		)
 		(property "Value" "LMV393"
-			(at 138.684 172.0851 0)
+			(at 143.51 174.244 0)
 			(effects
 				(font
-					(size 0.635 0.635)
+					(size 1.27 1.27)
 				)
-				(justify left)
 			)
 		)
@@
 		(pin "4"
 		)
+		(pin "9"
+		)
 		(instances
 			(project "Pinball Matrix board Rev 1"
@@
 	)
 	(symbol
+		(lib_name "LMV393_4")
 		(lib_id "Comparator:LMV393")
 		(at 129.54 170.18 0)
@@
 		(on_board yes)
 		(dnp no)
-		(fields_autoplaced yes)
 		(property "Reference" "U1"
-			(at 128.27 169.5449 0)
+			(at 127.762 170.18 0)
 			(effects
 				(font
 					(size 1.27 1.27)
 				)
-				(justify left)
 			)
 		)
 		(property "Value" "LMV393"
-			(at 128.27 171.45 0)
+			(at 121.92 155.702 0)
 			(effects
 				(font
-					(size 0.635 0.635)
+					(size 1.27 1.27)
 				)
-				(justify left)
+				(hide yes)
 			)
 		)
@@
 		(pin "4"
 		)
+		(pin "9"
+		)
 		(instances
 			(project ""
@@
 	)
 	(symbol
+		(lib_name "LMV393_5")
 		(lib_id "Comparator:LMV393")
 		(at 87.63 176.53 0)
@@
 		(dnp no)
 		(property "Reference" "U1"
-			(at 86.106 176.022 0)
+			(at 85.852 176.53 0)
 			(effects
 				(font
@@
 		)
 		(property "Value" "LMV393"
-			(at 90.17 180.594 0)
+			(at 88.138 181.864 0)
 			(effects
 				(font
@@
 		(pin "4"
 		)
+		(pin "9"
+		)
 		(instances
 			(project ""
@@
 			)
 		)
+		(pin "1"
+		)
 		(instances
 			(project "Pinball Matrix board Rev 1"
@@
 	)
 	(symbol
+		(lib_name "LMV393_3")
 		(lib_id "Comparator:LMV393")
 		(at 87.63 226.06 0)
@@
 		(pin "4"
 		)
+		(pin "9"
+		)
 		(instances
 			(project "Pinball Matrix board Rev 1"
@@
 	)
 	(symbol
+		(lib_name "LMV393_2")
 		(lib_id "Comparator:LMV393")
 		(at 87.63 250.19 0)
@@
 		(dnp no)
 		(property "Reference" "U2"
-			(at 85.852 250.19 0)
+			(at 86.106 249.682 0)
 			(effects
 				(font
@@
 		)
 		(property "Value" "LMV393"
-			(at 88.138 255.524 0)
+			(at 90.17 254.254 0)
 			(effects
 				(font
@@
 		(pin "4"
 		)
+		(pin "9"
+		)
 		(instances
 			(project "Pinball Matrix board Rev 1"
@@
 			)
 		)
-		(property "Footprint" "POWERSSO-16_STM"
+		(property "Footprint" "1My_Parts_ ICs:SOP50P600X148-17N"
 			(at 288.29 38.1 0)
 			(effects
@@
 		(pin "4"
 		)
-		(pin "EPAD"
+		(pin "17"
 		)
 		(pin "2"
@@
 	)
 	(symbol
+		(lib_name "MountingHole_2")
 		(lib_id "Mechanical:MountingHole")
 		(at 313.69 226.06 0)
@@
 			)
 		)
+		(pin "1"
+		)
 		(instances
 			(project "Pinball Matrix board Rev 1"
@@
 	)
 	(symbol
+		(lib_name "VNQ7E100AJTR_1")
 		(lib_id "1My_IC's:VNQ7E100AJTR")
 		(at 288.29 102.87 0)
@@
 			)
 		)
-		(property "Footprint" "POWERSSO-16_STM"
+		(property "Footprint" "1My_Parts_ ICs:SOP50P600X148-17N"
 			(at 288.29 102.87 0)
 			(effects
@@
 		(pin "4"
 		)
-		(pin "EPAD"
+		(pin "17"
 		)
 		(pin "2"
@@
 			)
 		)
-		(property "Footprint" "Through Hole,P=5.1mm"
+		(property "Footprint" "OptoDevice:R_LDR_7x6mm_P5.1mm_Vertical"
 			(at 55.88 31.75 0)
 			(effects
@@
 	)
 	(symbol
+		(lib_name "MountingHole_1")
 		(lib_id "Mechanical:MountingHole")
 		(at 313.69 220.98 0)
@@
 			)
 		)
+		(pin "1"
+		)
 		(instances
 			(project "Pinball Matrix board Rev 1"
@@
 					(unit 1)
 				)
+			)
+		)
+	)
+	(symbol
+		(lib_id "power:GND")
+		(at 313.69 236.22 0)
+		(unit 1)
+		(exclude_from_sim no)
+		(in_bom yes)
+		(on_board yes)
+		(dnp no)
+		(fields_autoplaced yes)
+		(property "Reference" "#PWR041"
+			(at 313.69 242.57 0)
+			(effects
+				(font
+					(size 1.27 1.27)
+				)
+				(hide yes)
+			)
+		)
+		(property "Value" "GND"
+			(at 313.69 241.3 0)
+			(effects
+				(font
+					(size 1.27 1.27)
+				)
+			)
+		)
+		(property "Footprint" ""
+			(at 313.69 236.22 0)
+			(effects
+				(font
+					(size 1.27 1.27)
+				)
+				(hide yes)
+			)
+		)
+		(property "Datasheet" ""
+			(at 313.69 236.22 0)
+			(effects
+				(font
+					(size 1.27 1.27)
+				)
+				(hide yes)
+			)
+		)
+		(property "Description" "Power symbol creates a global label with name \"GND\" , ground"
+			(at 313.69 236.22 0)
+			(effects
+				(font
+					(size 1.27 1.27)
+				)
+				(hide yes)
+			)
+		)
+		(pin "1"
+		)
+		(instances
+			(project ""
+				(path "/568ca592-389b-4e2e-8ed5-91d3bcea7500"
+					(reference "#PWR041")
+					(unit 1)
+				)
