File: hardware/Pinball Matrix board Rev 1.kicad_sch (KiCad schematic)
At the start: 155 parts, among them J1 B4B-XH-A, J2 B4B-XH-A, J3 Conn_01x13_Pin, J4 Conn_01x10_Pin, U1 LMV393, U2 LMV393, U3 ESP32-C6-DevKitM-Amazon, U4 74HC595D, U5 74HC595D, U6 VNQ7E100AJTR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

Commit message: Add files via upload
Parts:
- added 10mm1: ~, 1My_Parts_ Passive:10mm LOGO, symbol 1My Passive:TNES_Logo_10mm
- added D4: Yellow, PCM_JLCPCB:D_0805, symbol PCM_JLCPCB-Diodes:LED,0805,Yellow
- added R28: 3kΩ, PCM_JLCPCB:R_0805, symbol PCM_JLCPCB-Resistors:0805,3kΩ
- C16: value C_Polarized -> 330uf
- F2: footprint digikey-footprints:1206 -> PCM_JLCPCB:L_1206
- FB1, FB2, FB3, FB4, FB5, FB6, FB7: footprint PCM_JLCPCB:FB_0805 -> PCM_JLCPCB:L_1206
Connections:
- net +18vdc: now also D4.2
- net GND: now also R28.2
- new net: D4.1, R28.1
- no-connect marks 11 -> 10
Other:
- note added: "Output Connector"

Commit message: before PCB purchase
Parts:
- 10mm1, U3: now left out of the parts list
- F1: footprint OptoDevice:R_LDR_7x6mm_P5.1mm_Vertical -> 1My_Parts_ Passive:poly fuse
- H1, H2, H3: symbol Mechanical:MountingHole -> 1My Passive:MountingHole
- U8: value ~ -> OLED 256x128; now left out of the parts list
Connections:
- net GND: now also U1.9 (Epad), U2.9 (Epad)
Changed lines of the file:
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@@
 	)
 	(junction
+		(at 140.97 177.8)
+		(diameter 0)
+		(color 0 0 0 0)
+	)
+	(junction
 		(at 71.12 198.12)
 		(diameter 0)
@@
 	)
 	(junction
+		(at 129.54 177.8)
+		(diameter 0)
+		(color 0 0 0 0)
+	)
+	(junction
 		(at 72.39 128.27)
 		(diameter 0)
@@
 	(wire
 		(pts
-			(xy 127 177.8) (xy 133.35 177.8)
+			(xy 127 177.8) (xy 129.54 177.8)
 		)
 		(stroke
@@
 	(wire
 		(pts
+			(xy 129.54 177.8) (xy 133.35 177.8)
+		)
+		(stroke
+			(width 0)
+			(type default)
+		)
+	)
+	(wire
+		(pts
 			(xy 383.54 101.6) (xy 375.92 101.6)
 		)
@@
 	(wire
 		(pts
+			(xy 140.97 177.8) (xy 144.78 177.8)
+		)
+		(stroke
+			(width 0)
+			(type default)
+		)
+	)
+	(wire
+		(pts
 			(xy 54.61 223.52) (xy 71.12 223.52)
 		)
@@
 	(wire
 		(pts
-			(xy 138.43 177.8) (xy 144.78 177.8)
+			(xy 138.43 177.8) (xy 140.97 177.8)
 		)
 		(stroke
@@
 			)
 		)
-		(property "Datasheet" "https://www.lcsc.com/datasheet/lcsc_datasheet_2206010200_UNI-ROYAL-Uniroyal-Elec-0805W8F4702T5E_C17713.pdf"
+		(property "Datasheet" "https://www.lcsc.com/datasheet/lcsc_datasheet_2206010200_UNI-ROYAL-Uniroyal-Elec-0805W8F4701T5E_C17673.pdf"
 			(at 54.61 227.33 0)
 			(effects
@@
 		(exclude_from_sim no)
 		(in_bom yes)
-		(on_board no)
+		(on_board yes)
 		(dnp no)
 		(property "Reference" "R71"
@@
 			)
 		)
-		(property "Datasheet" "https://www.lcsc.com/datasheet/lcsc_datasheet_2206010200_UNI-ROYAL-Uniroyal-Elec-0805W8F4702T5E_C17713.pdf"
+		(property "Datasheet" "https://www.lcsc.com/datasheet/lcsc_datasheet_2206010200_UNI-ROYAL-Uniroyal-Elec-0805W8F4701T5E_C17673.pdf"
 			(at 54.61 177.8 0)
 			(effects
@@
 	)
 	(symbol
-		(lib_id "Mechanical:MountingHole")
+		(lib_id "1My Passive:MountingHole")
 		(at 313.69 231.14 0)
 		(unit 1)
@@
 		(fields_autoplaced yes)
 		(property "Reference" "H3"
-			(at 316.23 229.8699 0)
+			(at 317.5 229.8699 0)
 			(effects
 				(font
@@
 		)
 		(property "Value" "MountingHole"
-			(at 316.23 232.4099 0)
+			(at 317.5 232.4099 0)
 			(effects
 				(font
@@
 		(exclude_from_sim no)
 		(in_bom yes)
-		(on_board no)
+		(on_board yes)
 		(dnp no)
 		(property "Reference" "FB8"
@@
 			)
 		)
-		(property "Datasheet" "https://www.lcsc.com/datasheet/lcsc_datasheet_2206010200_UNI-ROYAL-Uniroyal-Elec-0805W8F4702T5E_C17713.pdf"
+		(property "Datasheet" "https://www.lcsc.com/datasheet/lcsc_datasheet_2206010200_UNI-ROYAL-Uniroyal-Elec-0805W8F4701T5E_C17673.pdf"
 			(at 55.88 251.46 0)
 			(effects
@@
 	)
 	(symbol
-		(lib_name "MountingHole_2")
-		(lib_id "Mechanical:MountingHole")
+		(lib_id "1My Passive:MountingHole")
 		(at 313.69 226.06 0)
 		(unit 1)
@@
 		(fields_autoplaced yes)
 		(property "Reference" "H2"
-			(at 316.23 224.7899 0)
+			(at 317.5 224.7899 0)
 			(effects
 				(font
@@
 		)
 		(property "Value" "MountingHole"
-			(at 316.23 227.3299 0)
+			(at 317.5 227.3299 0)
 			(effects
 				(font
@@
 		(unit 1)
 		(exclude_from_sim no)
-		(in_bom yes)
+		(in_bom no)
 		(on_board yes)
 		(dnp no)
@@
 		(exclude_from_sim no)
 		(in_bom yes)
-		(on_board no)
+		(on_board yes)
 		(dnp no)
 		(property "Reference" "C33"
@@
 			)
 		)
-		(property "Footprint" "OptoDevice:R_LDR_7x6mm_P5.1mm_Vertical"
+		(property "Footprint" "1My_Parts_ Passive:poly fuse"
 			(at 55.88 31.75 0)
 			(effects
@@
 	)
 	(symbol
-		(lib_name "MountingHole_1")
-		(lib_id "Mechanical:MountingHole")
+		(lib_id "1My Passive:MountingHole")
 		(at 313.69 220.98 0)
 		(unit 1)
@@
 		(fields_autoplaced yes)
 		(property "Reference" "H1"
-			(at 316.23 219.7099 0)
+			(at 317.5 219.7099 0)
 			(effects
 				(font
@@
 		)
 		(property "Value" "MountingHole"
-			(at 316.23 222.2499 0)
+			(at 317.5 222.2499 0)
 			(effects
 				(font
@@
 			)
 		)
-		(property "Datasheet" "https://www.lcsc.com/datasheet/lcsc_datasheet_2206010200_UNI-ROYAL-Uniroyal-Elec-0805W8F4702T5E_C17713.pdf"
+		(property "Datasheet" "https://www.lcsc.com/datasheet/lcsc_datasheet_2206010200_UNI-ROYAL-Uniroyal-Elec-0805W8F4701T5E_C17673.pdf"
 			(at 55.88 201.93 0)
 			(effects
@@
 		(unit 1)
 		(exclude_from_sim no)
-		(in_bom yes)
+		(in_bom no)
 		(on_board yes)
 		(dnp no)
@@
 			)
 		)
-		(property "Value" "~"
+		(property "Value" "OLED 256x128"
 			(at 186.69 46.9899 0)
 			(effects
@@
 		(unit 1)
 		(exclude_from_sim no)
-		(in_bom yes)
+		(in_bom no)
 		(on_board yes)
 		(dnp no)
