File: hardware/Pinball Matrix board Rev 1.kicad_pcb pre route.kicad_pcb (KiCad board)
At the start: 4 copper layers, 100 x 100 mm, 155 parts, among them J1 B4B-XH-A, J2 B4B-XH-A, J3 Conn_01x13_Pin, J4 Conn_01x10_Pin, U1 LMV393, U2 LMV393, U3 ESP32-C6-DevKitM-Amazon, U4 74HC595D, U5 74HC595D, U6 VNQ7E100AJTR, U7 VNQ7E100AJTR

Commit message: Add files via upload
Parts:
- removed REF**: 10mm LOGO, 1My_Parts_ Passive:10mm LOGO
- C16: value 330uf -> C_Polarized
- F2: footprint PCM_JLCPCB:L_1206 -> digikey-footprints:1206
- FB1, FB2, FB3, FB4, FB5, FB6, FB7: footprint PCM_JLCPCB:L_1206 -> PCM_JLCPCB:FB_0805
- moved R2 16.1 mm to (171.5, 64.2), turned to 90 degrees
- moved TP11 14.1 mm to (177.1, 63.8)
- moved TP12 14.1 mm to (180.5, 63.8)
- moved R1 10.6 mm to (168.6, 64.2), turned to 90 degrees
- moved C34 4.55 mm to (186.3, 75.1)
- moved F2 2.38 mm to (174.6, 54.2), turned to 90 degrees
- moved C24 2.05 mm to (127.8, 89.7), turned to 90 degrees
- moved C22 1.93 mm to (124.9, 89.7), turned to 90 degrees
- moved R65 1.41 mm to (106.0, 132.3), turned to -90 degrees
- moved C27 1.41 mm to (108.8, 132.3)
- moved FB2 1.41 mm to (103.6, 132.3)
- moved C15 0.91 mm to (129.3, 75.6)
- moved C23 0.84 mm to (125.3, 75.5)
- turned FB4 to -90 degrees
- turned R36 to 180 degrees
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- renumbered +5V to TP1, SDA to TP11, SCL to TP12, 3.3v to TP2, GPIO0 to TP3, GPIO1 to TP4, GPIO8 to TP5, GND to TP6, GPIO11 to TP7, GPIO12 to TP8, GPIO13 to TP9
Routing:
- net +3.3V: track 224.1 -> 0.00 mm, vias 1 -> 0
- net VCC_5V: track 138.6 -> 0.00 mm, vias 2 -> 0
- net GND: track 129.3 -> 0.00 mm, vias 25 -> 0
- net I²C SDA: track 79.2 -> 0.00 mm
- net I²C SCL: track 76.3 -> 0.00 mm, vias 1 -> 0
- net S_CLK: track 74.1 -> 0.00 mm, vias 2 -> 0
- net S_latch: track 64.7 -> 0.00 mm, vias 2 -> 0
- net SR /OE: track 62.2 -> 0.00 mm, vias 1 -> 0
- net LD3: track 60.0 -> 0.00 mm, vias 1 -> 0
- net Sw_Col_3: track 58.6 -> 0.00 mm, vias 1 -> 0
- net Sw_Col_2: track 58.4 -> 0.00 mm, vias 1 -> 0
- net Sw_Col_1: track 58.2 -> 0.00 mm, vias 1 -> 0
- net Sw_Col_0: track 58.0 -> 0.00 mm, vias 1 -> 0
- net Fault_RST 5-8: track 56.5 -> 0.00 mm, vias 2 -> 0
- net Row_2: track 55.8 -> 0.00 mm, vias 2 -> 0
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- removed copper zone on B.Cu, net GND
- removed copper zone on F.Cu, net GND
Other:
- copper layers 4 -> 2
- board text removed: "Antenna"
- board text removed: "ESP32-C6-DevKitM-Amazon"
- board text removed: "P Forche TNES LLC 2026 Rev 0"
