File: hardware/Pinball Matrix board Rev 1_routed power.kicad_pcb (KiCad board)
At the start: 4 copper layers, 100 x 100 mm, 155 parts, among them J1 B4B-XH-A, J2 B4B-XH-A, J3 Conn_01x13_Pin, J4 Conn_01x10_Pin, U1 LMV393, U2 LMV393, U3 ESP32-C6-DevKitM-Amazon, U4 74HC595D, U5 74HC595D, U6 VNQ7E100AJTR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

Commit message: Add files via upload
Parts:
- removed REF**: 10mm LOGO, 1My_Parts_ Passive:10mm LOGO
Routing:
- net Net-(R14-Pad2): track 30.0 -> 46.4 mm, vias 2 -> 3
- net +5V: track 53.3 -> 54.9 mm
- net SW_2: track 31.9 -> 33.4 mm
Other:
- board text removed: "ESP32-C6-DevKitM-Amazon"
- board text removed: "P Forche TNES LLC 2026 Rev 0"
